File: pcb/name-badge-sao/name-badge-sao.kicad_sch (KiCad schematic)
At the start: 109 parts, among them J1 USB_C_Receptacle_USB2.0, J2 Conn_01x02, SW1 SW_SPDT, U1 IS31FL3731-QF, U2 SAMD21_MOD, U3 W25Q32JVSS, U4 TP4057

Commit message: Moving to an all-new circuit design (normal matrix, no charlieplexing) with a new MCU, because why not change everything?
Parts:
- removed C1: 100n, Capacitor_SMD:C_0603_1608Metric, symbol chipsetter-badge-sao-eagle-import:C-USC0603
- removed C5: 10u, Capacitor_SMD:C_0805_2012Metric, symbol chipsetter-badge-sao-eagle-import:C-USC0603
- removed C6: 1u, Capacitor_SMD:C_0603_1608Metric, symbol chipsetter-badge-sao-eagle-import:C-USC0603
- removed J1: USB_C_Receptacle_USB2.0, Connector_USB:USB_C_Receptacle_HRO_TYPE-C-31-M-12, symbol Connector:USB_C_Receptacle_USB2.0
- removed J2: Conn_01x02, Connector_PinHeader_2.00mm:PinHeader_1x02_P2.00mm_Vertical, symbol Connector_Generic:Conn_01x02
- removed LED1, LED10, LED11, LED12, LED13, LED14, LED15, LED16, LED17, LED18, LED19, LED2, LED20, LED21, LED22, LED23, LED24, LED25, LED26, LED27, LED28, LED29, LED3, LED30, LED31, LED32, LED33, LED34, LED35, LED36, LED37, LED38, LED39, LED4, LED40, LED41, LED42, LED43, LED44, LED45, LED46, LED47, LED48, LED49, LED5, LED50, LED51, LED52, LED53, LED54, LED55, LED56, LED57, LED58, LED59, LED6, LED60, LED61, LED62, LED63, LED64, LED65, LED66, LED67, LED68, LED69, LED7, LED70, LED71, LED72, LED73, LED74, LED75, LED76, LED77, LED78, LED79, LED8, LED80, LED81, LED82, LED9: LED, LED_SMD:LED_0603_1608Metric, symbol Device:LED
- removed R1, R2, R9: 10K, Resistor_SMD:R_0603_1608Metric, symbol chipsetter-badge-sao-eagle-import:R-US_R0603
- removed R3, R4: 5.1K, Resistor_SMD:R_0603_1608Metric, symbol chipsetter-badge-sao-eagle-import:R-US_R0603
- removed R5, R6: DNP, Resistor_SMD:R_0603_1608Metric, symbol chipsetter-badge-sao-eagle-import:R-US_R0603
- removed R7, R8: 1K, Resistor_SMD:R_0603_1608Metric, symbol chipsetter-badge-sao-eagle-import:R-US_R0603
- removed SW1: SW_SPDT, Button_Switch_SMD:SW_SPDT_PCM12, symbol Switch:SW_SPDT
- removed U1: IS31FL3731-QF, Package_DFN_QFN:QFN-28-1EP_4x4mm_P0.4mm_EP2.3x2.3mm, symbol Driver_LED:IS31FL3731-QF
- removed U2: SAMD21_MOD, hcc_mod:SAMD_HCC_G_FOOT, symbol samd_hcc_mod:SAMD21_MOD
- removed U3: W25Q32JVSS, Package_SO:SOIC-8_5.23x5.23mm_P1.27mm, symbol Memory_Flash:W25Q32JVSS
- removed U4: TP4057, Package_TO_SOT_SMD:SOT-23-6, symbol TP4057:TP4057
- added D1, D10, D100, D101, D102, D103, D104, D105, D106, D107, D108, D109, D11, D110, D111, D112, D113, D114, D115, D116, D117, D118, D119, D12, D120, D121, D122, D123, D124, D125, D126, D127, D128, D13, D14, D15, D16, D17, D18, D19, D2, D20, D21, D22, D23, D24, D25, D26, D27, D28, D29, D3, D30, D31, D32, D33, D34, D35, D36, D37, D38, D39, D4, D40, D41, D42, D43, D44, D45, D46, D47, D48, D49, D5, D50, D51, D52, D53, D54, D55, D56, D57, D58, D59, D6, D60, D61, D62, D63, D64, D65, D66, D67, D68, D69, D7, D70, D71, D72, D73, D74, D75, D76, D77, D78, D79, D8, D80, D81, D82, D83, D84, D85, D86, D87, D88, D89, D9, D90, D91, D92, D93, D94, D95, D96, D97, D98, D99: LED, LED_SMD:LED_0603_1608Metric, symbol Device:LED
- added Q1, Q10, Q11, Q12, Q13, Q14, Q15, Q16, Q2, Q3, Q4, Q5, Q6, Q7, Q8, Q9: MMBT3904, Package_TO_SOT_SMD:SOT-23, symbol Transistor_BJT:MMBT3904
- added R10, R11, R14, R15, R16, R17, R18, R19, R20, R21, R22, R23, R24, R25, R26, R27: 1K, Resistor_SMD:R_0603_1608Metric, symbol Device:R
- added R28, R29, R30, R31, R32, R33, R34, R35: 100, Resistor_SMD:R_0603_1608Metric, symbol Device:R
- added U5: STM32F030C8Tx, Package_QFP:LQFP-48_7x7mm_P0.5mm, symbol MCU_ST_STM32F0:STM32F030C8Tx
Connections:
- net +3V3: now also U5.1 (VDD), U5.24 (VDD), U5.48 (VDD), U5.9 (VDDA)
- net GND: now also Q1.2 (E), Q10.2 (E), Q11.2 (E), Q12.2 (E), Q13.2 (E), Q14.2 (E), Q15.2 (E), Q16.2 (E), Q2.2 (E), Q3.2 (E), Q4.2 (E), Q5.2 (E), Q6.2 (E), Q7.2 (E), Q8.2 (E), Q9.2 (E), U5.23 (VSS), U5.47 (VSS), U5.8 (VSSA)
- net SCL: now also U5.6 (PF1)
- net SDA: now also U5.5 (PF0)
- new net: D73.1 (K), D74.1 (K), D75.1 (K), D76.1 (K), D77.1 (K), D78.1 (K), D79.1 (K), D80.1 (K), Q10.3 (C)
- new net: D102.2 (A), D110.2 (A), D118.2 (A), D126.2 (A), D14.2 (A), D22.2 (A), D30.2 (A), D38.2 (A), D46.2 (A), D54.2 (A), D6.2 (A), D62.2 (A), D70.2 (A), D78.2 (A), D86.2 (A), D94.2 (A), R33.1
- new net: D33.1 (K), D34.1 (K), D35.1 (K), D36.1 (K), D37.1 (K), D38.1 (K), D39.1 (K), D40.1 (K), Q5.3 (C)
- new net: D1.2 (A), D105.2 (A), D113.2 (A), D121.2 (A), D17.2 (A), D25.2 (A), D33.2 (A), D41.2 (A), D49.2 (A), D57.2 (A), D65.2 (A), D73.2 (A), D81.2 (A), D89.2 (A), D9.2 (A), D97.2 (A), R28.1
- new net: D25.1 (K), D26.1 (K), D27.1 (K), D28.1 (K), D29.1 (K), D30.1 (K), D31.1 (K), D32.1 (K), Q4.3 (C)
- new net: D57.1 (K), D58.1 (K), D59.1 (K), D60.1 (K), D61.1 (K), D62.1 (K), D63.1 (K), D64.1 (K), Q8.3 (C)
- new net: D10.2 (A), D106.2 (A), D114.2 (A), D122.2 (A), D18.2 (A), D2.2 (A), D26.2 (A), D34.2 (A), D42.2 (A), D50.2 (A), D58.2 (A), D66.2 (A), D74.2 (A), D82.2 (A), D90.2 (A), D98.2 (A), R29.1
- new net: D17.1 (K), D18.1 (K), D19.1 (K), D20.1 (K), D21.1 (K), D22.1 (K), D23.1 (K), D24.1 (K), Q3.3 (C)
- new net: D101.2 (A), D109.2 (A), D117.2 (A), D125.2 (A), D13.2 (A), D21.2 (A), D29.2 (A), D37.2 (A), D45.2 (A), D5.2 (A), D53.2 (A), D61.2 (A), D69.2 (A), D77.2 (A), D85.2 (A), D93.2 (A), R32.1
- new net: D81.1 (K), D82.1 (K), D83.1 (K), D84.1 (K), D85.1 (K), D86.1 (K), D87.1 (K), D88.1 (K), Q11.3 (C)
- new net: D107.2 (A), D11.2 (A), D115.2 (A), D123.2 (A), D19.2 (A), D27.2 (A), D3.2 (A), D35.2 (A), D43.2 (A), D51.2 (A), D59.2 (A), D67.2 (A), D75.2 (A), D83.2 (A), D91.2 (A), D99.2 (A), R30.1
- new net: Q7.1 (B), R18.2
- new net: D49.1 (K), D50.1 (K), D51.1 (K), D52.1 (K), D53.1 (K), D54.1 (K), D55.1 (K), D56.1 (K), Q7.3 (C)
- new net: Q5.1 (B), R16.2
- new net: D103.2 (A), D111.2 (A), D119.2 (A), D127.2 (A), D15.2 (A), D23.2 (A), D31.2 (A), D39.2 (A), D47.2 (A), D55.2 (A), D63.2 (A), D7.2 (A), D71.2 (A), D79.2 (A), D87.2 (A), D95.2 (A), R34.1
- new net: D105.1 (K), D106.1 (K), D107.1 (K), D108.1 (K), D109.1 (K), D110.1 (K), D111.1 (K), D112.1 (K), Q14.3 (C)
- new net: D121.1 (K), D122.1 (K), D123.1 (K), D124.1 (K), D125.1 (K), D126.1 (K), D127.1 (K), D128.1 (K), Q16.3 (C)
- new net: D113.1 (K), D114.1 (K), D115.1 (K), D116.1 (K), D117.1 (K), D118.1 (K), D119.1 (K), D120.1 (K), Q15.3 (C)
- new net: D100.2 (A), D108.2 (A), D116.2 (A), D12.2 (A), D124.2 (A), D20.2 (A), D28.2 (A), D36.2 (A), D4.2 (A), D44.2 (A), D52.2 (A), D60.2 (A), D68.2 (A), D76.2 (A), D84.2 (A), D92.2 (A), R31.1
- new net: D100.1 (K), D101.1 (K), D102.1 (K), D103.1 (K), D104.1 (K), D97.1 (K), D98.1 (K), D99.1 (K), Q13.3 (C)
- new net: D65.1 (K), D66.1 (K), D67.1 (K), D68.1 (K), D69.1 (K), D70.1 (K), D71.1 (K), D72.1 (K), Q9.3 (C)
- new net: D41.1 (K), D42.1 (K), D43.1 (K), D44.1 (K), D45.1 (K), D46.1 (K), D47.1 (K), D48.1 (K), Q6.3 (C)
- new net: D104.2 (A), D112.2 (A), D120.2 (A), D128.2 (A), D16.2 (A), D24.2 (A), D32.2 (A), D40.2 (A), D48.2 (A), D56.2 (A), D64.2 (A), D72.2 (A), D8.2 (A), D80.2 (A), D88.2 (A), D96.2 (A), R35.1
- new net: D1.1 (K), D2.1 (K), D3.1 (K), D4.1 (K), D5.1 (K), D6.1 (K), D7.1 (K), D8.1 (K), Q1.3 (C)
- new net: Q2.1 (B), R11.2
- new net: D10.1 (K), D11.1 (K), D12.1 (K), D13.1 (K), D14.1 (K), D15.1 (K), D16.1 (K), D9.1 (K), Q2.3 (C)
- new net: Q10.1 (B), R21.2
- new net: Q6.1 (B), R17.2
- new net: D89.1 (K), D90.1 (K), D91.1 (K), D92.1 (K), D93.1 (K), D94.1 (K), D95.1 (K), D96.1 (K), Q12.3 (C)
- new net: Q8.1 (B), R19.2
- new net: Q13.1 (B), R24.2
- new net: Q4.1 (B), R15.2
- new net: Q11.1 (B), R22.2
- new net: Q14.1 (B), R25.2
- new net: Q15.1 (B), R26.2
- new net: Q12.1 (B), R23.2
- new net: Q3.1 (B), R14.2
- new net: Q9.1 (B), R20.2
- new net: Q1.1 (B), R10.2
- new net: Q16.1 (B), R27.2
- new net COL0: R10.1, U5.26 (PB13)
- new net COL1: R11.1, U5.25 (PB12)
- new net COL10: R22.1, U5.45 (PB8)
- new net COL11: R23.1, U5.43 (PB7)
- new net COL12: R24.1, U5.42 (PB6)
- new net COL13: R25.1, U5.41 (PB5)
- new net COL14: R26.1, U5.40 (PB4)
- new net COL15: R27.1, U5.39 (PB3)
- new net COL2: R14.1, U5.22 (PB11)
- new net COL3: R15.1, U5.21 (PB10)
- new net COL4: R16.1, U5.20 (PB2)
- new net COL5: R17.1, U5.19 (PB1)
- new net COL6: R18.1, U5.18 (PB0)
- new net COL7: R19.1, U5.27 (PB14)
- new net COL8: R20.1, U5.28 (PB15)
- new net COL9: R21.1, U5.46 (PB9)
- new net ROW0: R28.2, U5.17 (PA7)
- new net ROW1: R29.2, U5.16 (PA6)
- new net ROW2: R30.2, U5.15 (PA5)
- new net ROW3: R31.2, U5.14 (PA4)
- new net ROW4: R32.2, U5.13 (PA3)
- new net ROW5: R33.2, U5.12 (PA2)
- new net ROW6: R34.2, U5.11 (PA1)
- new net ROW7: R35.2, U5.10 (PA0)
- new net SWCLK: U5.37 (PA14)
- new net SWDIO: U5.34 (PA13)
- new net ~{RESET}: U5.7 (NRST)
- no-connect marks 3 -> 0
Other:
- moved on the sheet: C2, C3, C4, R12, R13, S1, S2

Commit message: I think that's an SAO
Parts:
- removed SAO1: AVR-ISP-6SMD, Connector_IDC:IDC-Header_2x03_P2.54mm_Vertical, symbol chipsetter-badge-sao-eagle-import:AVR-ISP-6SMD
- added J1: Conn_02x03_Odd_Even, Connector_IDC:IDC-Header_2x03_P2.54mm_Vertical_SMD, symbol Connector_Generic:Conn_02x03_Odd_Even
- added J2: BOOT0, TestPoint:TestPoint_Pad_1.5x1.5mm, symbol Connector_Generic:Conn_01x01
- added J3: RESET, TestPoint:TestPoint_Pad_1.5x1.5mm, symbol Connector_Generic:Conn_01x01
- added J4: SWDIO, TestPoint:TestPoint_Pad_1.5x1.5mm, symbol Connector_Generic:Conn_01x01
- added J5: SWCLK, TestPoint:TestPoint_Pad_1.5x1.5mm, symbol Connector_Generic:Conn_01x01
- added R1: 10K, Resistor_SMD:R_0603_1608Metric, symbol Device:R
Connections:
- net RESET is gone; now on net ~{RESET}: R13.1, S2.2 (S)
- net +3V3: now also J1.1 (Pin_1), R1.2
- net BUTTON: now also U5.29 (PA8)
- net GND: now also J1.2 (Pin_2)
- net SCL: now also J1.4 (Pin_4)
- net SDA: now also J1.3 (Pin_3)
- net SWCLK: now also J5.1 (Pin_1)
- net SWDIO: now also J4.1 (Pin_1)
- net ~{RESET}: now also J3.1 (Pin_1)
- net UART_RX: now reaches U5.30 (PA9)
- net UART_RX: now also J1.5 (Pin_5)
- net UART_TX: now reaches U5.31 (PA10)
- net UART_TX: now also J1.6 (Pin_6)
- net at U5.44 (BOOT0): now also J2.1 (Pin_1), R1.1
